File: _autosave-IC.kicad_sch (KiCad schematic)
At the start: 24 parts, among them IC1 BTS722204ESAXUMA1

Commit message: Finished schematic
Added UCB C connection
Added CAN
Power ICs schematic fixed
Parts:
- R16, R17, R18: value 1.2k -> 330
