File: LEDs.kicad_sch (KiCad schematic)
At the start: 8 parts

Commit message: Footprint changes + started PCB
Parts:
- R1, R2, R3, R4: value 130 -> 150; footprint Resistor_SMD:R_0603_1608Metric -> Resistor_SMD:R_0603_1608Metric_Pad0.98x0.95mm_HandSolder; m CRCW0603330RFKEBC -> WR06X1500FTL
Connections:
- net at D1.2 (A): now also R3.2; no longer R1.2
- net at D3.2 (A): now also R1.2; no longer R3.2
