File: Power.kicad_sch (KiCad schematic)
At the start: 24 parts, among them U2 LD1117S33TR_SOT223, U3 LM2675M-5.0/NOPB

Commit message: Minor fixes
Connections:
- net +5V: now also F1.1
Other:
- moved on the sheet: C27, C28, D10, D11, F1

Commit message: Footprint changes + started PCB
Parts:
- C27: footprint (none) -> Capacitor_SMD:CP_Elec_4x4.5; Mouser (none) -> https://www.mouser.pl/ProductDetail/Wurth-Elektronik/865080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
- C28: footprint (none) -> Capacitor_SMD:C_0603_1608Metric_Pad1.08x0.95mm_HandSolder
- D10: footprint (none) -> Diode_SMD:D_SMA; Mouser (none) -> https://www.mouser.pl/ProductDetail/Taiwan-Semiconductor/SS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
- D11: footprint (none) -> Diode_SMD:D_SOD-123; Mouser  (none) -> https://www.mouser.pl/ProductDetail/Diodes-Incorporated/MMS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; model  (none) -> MMSZ5233B-7-F
- F1: footprint (none) -> Fuse:Fuse_1206_3216Metric_Pad1.42x1.75mm_HandSolder; Mouser (none) -> https://www.mouser.pl/ProductDetail/Eaton-Electronics/PTS12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
Changed lines of the file:
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@@
 			)
 		)
-		(property "Footprint" ""
+		(property "Footprint" "Fuse:Fuse_1206_3216Metric_Pad1.42x1.75mm_HandSolder"
 			(at 227.33 96.52 0)
 			(effects
@@
 			)
 		)
-		(property "Datasheet" "~"
+		(property "Datasheet" "https://www.mouser.pl/datasheet/2/87/eaton_pts1206_6_60_volt_dc_surface_mount_resettabl-1608737.pdf"
 			(at 228.6 91.44 0)
 			(effects
@@
 		)
 		(property "Description" "Resettable fuse, polymeric positive temperature coefficient, small symbol"
+			(at 228.6 91.44 0)
+			(effects
+				(font
+					(size 1.27 1.27)
+				)
+				(hide yes)
+			)
+		)
+		(property "Mouser" "https://www.mouser.pl/ProductDetail/Eaton-Electronics/PTS120615V050?qs=QmibqUXyDhQpLmnP4WG6Mg%3D%3D"
 			(at 228.6 91.44 0)
 			(effects
@@
 			)
 		)
-		(property "Footprint" ""
+		(property "Footprint" "Diode_SMD:D_SMA"
 			(at 250.19 91.44 90)
 			(effects
@@
 			)
 		)
-		(property "Datasheet" "~"
+		(property "Datasheet" "https://services.taiwansemi.com/storage/resources/datasheet/SS12%20SERIES_R2305.pdf"
 			(at 250.19 91.44 90)
 			(effects
@@
 			)
 		)
-		(property "Description" "Schottky diode, small symbol"
+		(property "Description" "SS12 "
 			(at 250.19 91.44 0)
+			(effects
+				(font
+					(size 1.27 1.27)
+				)
+				(hide yes)
+			)
+		)
+		(property "Mouser" "https://www.mouser.pl/ProductDetail/Taiwan-Semiconductor/SS12?qs=JV7lzlMm3yJmZoP3vIhYAg%3D%3D"
+			(at 250.19 91.44 90)
 			(effects
 				(font
@@
 			)
 		)
-		(property "Footprint" ""
+		(property "Footprint" "Capacitor_SMD:C_0603_1608Metric_Pad1.08x0.95mm_HandSolder"
 			(at 240.03 99.06 0)
 			(effects
@@
 			)
 		)
-		(property "Footprint" ""
+		(property "Footprint" "Capacitor_SMD:CP_Elec_4x4.5"
 			(at 250.19 99.06 0)
 			(effects
@@
 			)
 		)
-		(property "Datasheet" "~"
+		(property "Datasheet" "https://www.we-online.com/components/products/datasheet/865080340003.pdf"
 			(at 250.19 99.06 0)
 			(effects
@@
 			)
 		)
-		(property "Description" "Polarized capacitor, small symbol"
+		(property "Description" "865080340003"
+			(at 250.19 99.06 0)
+			(effects
+				(font
+					(size 1.27 1.27)
+				)
+				(hide yes)
+			)
+		)
+		(property "Mouser" "https://www.mouser.pl/ProductDetail/Wurth-Elektronik/865080340003?qs=sGAEpiMZZMvwFf0viD3Y3aZipiehufnXiBteln9xyMrx1HfsRhyD8A%3D%3D"
 			(at 250.19 99.06 0)
 			(effects
@@
 			)
 		)
-		(property "Footprint" ""
+		(property "Footprint" "Diode_SMD:D_SOD-123"
 			(at 228.6 99.06 0)
 			(effects
@@
 			)
 		)
-		(property "Datasheet" "~"
+		(property "Datasheet" "https://www.mouser.pl/datasheet/2/115/DIOD_S_A0003550771_1-2542306.pdf"
 			(at 228.6 99.06 0)
 			(effects
@@
 			(effects
 				(font
+					(size 1.27 1.27)
+				)
+				(hide yes)
+			)
+		)
+		(property "model " "MMSZ5233B-7-F "
+			(at 228.6 99.06 90)
+			(effects
+				(font
+					(size 1.27 1.27)
+				)
+				(hide yes)
+			)
+		)
+		(property "Mouser " "https://www.mouser.pl/ProductDetail/Diodes-Incorporated/MMSZ5233B-7-F?qs=y%252B91MvA1s7t7mx7mwqyIpQ%3D%3D"
+			(at 228.6 99.06 90)
+			(effects
+				(font

Commit message: Minor changes
Parts:
- C27: value 22uF -> 22u
- C28: value 1uF -> 1u
Changed lines of the file:
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@@
 		(fields_autoplaced yes)
 		(property "Reference" "C28"
-			(at 237.49 97.7962 0)
-			(effects
-				(font
-					(size 1.27 1.27)
-				)
-				(justify left)
-			)
-		)
-		(property "Value" "1uF"
-			(at 237.49 100.3362 0)
-			(effects
-				(font
-					(size 1.27 1.27)
-				)
-				(justify left)
+			(at 242.57 97.7962 0)
+			(effects
+				(font
+					(size 1.27 1.27)
+				)
+				(justify right)
+			)
+		)
+		(property "Value" "1u"
+			(at 242.57 100.3362 0)
+			(effects
+				(font
+					(size 1.27 1.27)
+				)
+				(justify right)
 			)
 		)
@@
 			)
 		)
-		(property "Value" "22uF"
+		(property "Value" "22u"
 			(at 252.73 99.7838 0)
 			(effects

Commit message: Layout done
Added layout
Parts:
- renumbered Dr1 to D8
Changed lines of the file:
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@@
+	)
+	(junction
+		(at 162.56 120.65)
+		(diameter 0)
+		(color 0 0 0 0)
+	)
+	(junction
+		(at 58.42 45.72)
+		(diameter 0)
+		(color 0 0 0 0)
+	)
+	(junction
+		(at 137.16 135.89)
+		(diameter 0)
+		(color 0 0 0 0)
+	)
+	(junction
+		(at 123.19 69.85)
+		(diameter 0)
+		(color 0 0 0 0)
+	)
+	(junction
+		(at 153.67 135.89)
+		(diameter 0)
+		(color 0 0 0 0)
+	)
+	(junction
+		(at 138.43 91.44)
+		(diameter 0)
+		(color 0 0 0 0)
 	)
 	(junction
 		(at 250.19 93.98)
-		(diameter 0)
-		(color 0 0 0 0)
-	)
-	(junction
-		(at 162.56 120.65)
-		(diameter 0)
-		(color 0 0 0 0)
-	)
-	(junction
-		(at 58.42 45.72)
-		(diameter 0)
-		(color 0 0 0 0)
-	)
-	(junction
-		(at 137.16 135.89)
-		(diameter 0)
-		(color 0 0 0 0)
-	)
-	(junction
-		(at 123.19 69.85)
-		(diameter 0)
-		(color 0 0 0 0)
-	)
-	(junction
-		(at 153.67 135.89)
-		(diameter 0)
-		(color 0 0 0 0)
-	)
-	(junction
-		(at 138.43 91.44)
 		(diameter 0)
 		(color 0 0 0 0)
@@
 	)
 	(symbol
-		(lib_id "Device:D_Schottky_Small")
-		(at 250.19 91.44 270)
-		(mirror x)
-		(unit 1)
-		(exclude_from_sim no)
-		(in_bom yes)
-		(on_board yes)
-		(dnp no)
-		(property "Reference" "D10"
-			(at 247.65 90.4239 90)
-			(effects
-				(font
-					(size 1.27 1.27)
-				)
-				(justify right)
-			)
-		)
-		(property "Value" "0.1/1A"
-			(at 247.65 92.9639 90)
-			(effects
-				(font
-					(size 1.27 1.27)
-				)
-				(justify right)
-			)
-		)
-		(property "Footprint" "Diode_SMD:D_SMA"
-			(at 250.19 91.44 90)
-			(effects
-				(font
-					(size 1.27 1.27)
-				)
-				(hide yes)
-			)
-		)
-		(property "Datasheet" "https://services.taiwansemi.com/storage/resources/datasheet/SS12%20SERIES_R2305.pdf"
-			(at 250.19 91.44 90)
-			(effects
-				(font
-					(size 1.27 1.27)
-				)
-				(hide yes)
-			)
-		)
-		(property "Description" "SS12 "
-			(at 250.19 91.44 0)
-			(effects
-				(font
-					(size 1.27 1.27)
-				)
-				(hide yes)
-			)
-		)
-		(property "Mouser" "https://www.mouser.pl/ProductDetail/Taiwan-Semiconductor/SS12?qs=JV7lzlMm3yJmZoP3vIhYAg%3D%3D"
-			(at 250.19 91.44 90)
-			(effects
-				(font
-					(size 1.27 1.27)
-				)
-				(hide yes)
-			)
-		)
-		(pin "1"
-		)
-		(pin "2"
-		)
-		(instances
-			(project ""
-				(path "/b652b05a-4e3d-4ad1-b032-18886abe7d45/5554ce6e-235b-4b58-a8ae-0c0f8daf2a24"
-					(reference "D10")
-					(unit 1)
-				)
-			)
-		)
-	)
-	(symbol
 		(lib_id "Device:C_Small")
 		(at 240.03 99.06 0)
@@
 				(path "/b652b05a-4e3d-4ad1-b032-18886abe7d45/5554ce6e-235b-4b58-a8ae-0c0f8daf2a24"
 					(reference "C27")
+					(unit 1)
+				)
+			)
+		)
+	)
+	(symbol
+		(lib_id "Device:D_Schottky_Small")
+		(at 250.19 91.44 270)
+		(mirror x)
+		(unit 1)
+		(exclude_from_sim no)
+		(in_bom yes)
+		(on_board yes)
+		(dnp no)
+		(property "Reference" "D10"
+			(at 247.65 90.4239 90)
+			(effects
+				(font
+					(size 1.27 1.27)
+				)
+				(justify right)
+			)
+		)
+		(property "Value" "0.1/1A"
+			(at 247.65 92.9639 90)
+			(effects
+				(font
+					(size 1.27 1.27)
+				)
+				(justify right)
+			)
+		)
+		(property "Footprint" "Diode_SMD:D_SMA"
+			(at 250.19 91.44 90)
+			(effects
+				(font
+					(size 1.27 1.27)
+				)
+				(hide yes)
+			)
+		)
+		(property "Datasheet" "https://services.taiwansemi.com/storage/resources/datasheet/SS12%20SERIES_R2305.pdf"
+			(at 250.19 91.44 90)
+			(effects
+				(font
+					(size 1.27 1.27)
+				)
+				(hide yes)
+			)
+		)
+		(property "Description" "SS12 "
+			(at 250.19 91.44 0)
+			(effects
+				(font
+					(size 1.27 1.27)
+				)
+				(hide yes)
+			)
+		)
+		(property "Mouser" "https://www.mouser.pl/ProductDetail/Taiwan-Semiconductor/SS12?qs=JV7lzlMm3yJmZoP3vIhYAg%3D%3D"
+			(at 250.19 91.44 90)
+			(effects
+				(font
+					(size 1.27 1.27)
+				)
+				(hide yes)
+			)
+		)
+		(pin "1"
+		)
+		(pin "2"
+		)
+		(instances
+			(project "PUTM_EV_PDMv2_2024"
+				(path "/b652b05a-4e3d-4ad1-b032-18886abe7d45/5554ce6e-235b-4b58-a8ae-0c0f8daf2a24"
+					(reference "D10")
 					(unit 1)
 				)
@@
 		(dnp no)
 		(fields_autoplaced yes)
-		(property "Reference" "Dr1"
-			(at 60.96 60.0075 90)
+		(property "Reference" "D8"
+			(at 60.96 60.0074 90)
 			(effects
 				(font
@@
 		)
 		(property "Value" "SS34ALH"
-			(at 60.96 62.5475 90)
+			(at 60.96 62.5474 90)
 			(effects
 				(font
@@
 			(project "PUTM_EV_PDMv2_2024"
 				(path "/b652b05a-4e3d-4ad1-b032-18886abe7d45/5554ce6e-235b-4b58-a8ae-0c0f8daf2a24"
-					(reference "Dr1")
+					(reference "D8")
 					(unit 1)
 				)
