File: hardware/ic_3.kicad_sch (KiCad schematic)
At the start: 24 parts, among them IC4 BTS722204ESAXUMA1

Commit message: new pcb layout & can coppied from steeringwheel
Parts:
- renumbered C53 to C52, C54 to C53, C55 to C54, C56 to C55, C57 to C56, C58 to C57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
Connections:
- net PC3_GND: now reaches C54.2, C55.1, IC4.1 (GND), R69.2
- net VDD: now reaches C55.2, IC4.2 (VDD), R59.2
- net LHI: now reaches IC4.7 (LHI), R57.2
- net R_IS_PROT: now reaches D15.1 (K), R56.2, R58.1
